File: thaco-led-54x930.kicad_pcb (KiCad board)
At the start: 2 copper layers, 930 x 54 mm, 94 parts, among them P1 CONN_01X03, P5 CONN_01X03, P6 CONN_01X03

Commit message: project finish
Parts:
- added REF**: hole, holemoi:hole, F.Cu at (156.2, 595.0)
- added REF**: hole, holemoi:hole, F.Cu at (388.8, 595.0)
- added REF**: hole, holemoi:hole, F.Cu at (621.2, 595.0)
- added REF**: hole, holemoi:hole, F.Cu at (853.8, 595.0)
Routing:
- net GND: track 3004.2 -> 3021.7 mm
- added copper zone on F.Cu, net GND
Changed lines of the file:
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@@
-(kicad_pcb (version 4) (host pcbnew 4.0.2+e4-6225~38~ubuntu16.04.1-stable)
+(kicad_pcb (version 4) (host pcbnew 4.0.2-stable)
   (general
     (links 263)
-    (no_connects 23)
-    (area 18.858251 547.15 975.406251 622.075001)
+    (no_connects 6)
+    (area 18.858251 539.5 975.406251 622.075001)
     (thickness 1.6)
-    (drawings 7)
-    (tracks 404)
+    (drawings 9)
+    (tracks 414)
     (zones 0)
-    (modules 94)
+    (modules 98)
     (nets 196)
   )
@@
     (pad_to_mask_clearance 0.2)
     (aux_axis_origin 0 0)
-    (grid_origin 40 622)
-    (visible_elements FFFFFF7F)
+    (grid_origin 505 595)
+    (visible_elements 7FFFFFFF)
     (pcbplotparams
-      (layerselection 0x00030_80000001)
+      (layerselection 0x010aa_00000001)
       (usegerberextensions false)
       (excludeedgelayer true)
@@
       (outputformat 1)
       (mirror false)
-      (drillshape 1)
+      (drillshape 0)
       (scaleselection 1)
-      (outputdirectory ""))
+      (outputdirectory gerber/))
   )
   (net 0 "")
@@
     )
   )
+  (module holemoi:hole (layer F.Cu)
+    (at 156.25 595)
+    (fp_text reference REF** (at 0 0.5) (layer F.SilkS)
+      (effects (font (size 1 1) (thickness 0.15)))
+    )
+    (fp_text value hole (at 0 -0.5) (layer F.Fab)
+      (effects (font (size 1 1) (thickness 0.15)))
+    )
+    (pad 1 thru_hole circle (at 0 0) (size 3 3) (drill 3) (layers *.Cu *.Mask F.SilkS))
+  )
+  (module holemoi:hole (layer F.Cu)
+    (at 388.75 595)
+    (fp_text reference REF** (at 0 0.5) (layer F.SilkS)
+      (effects (font (size 1 1) (thickness 0.15)))
+    )
+    (fp_text value hole (at 0 -0.5) (layer F.Fab)
+      (effects (font (size 1 1) (thickness 0.15)))
+    )
+    (pad 1 thru_hole circle (at 0 0) (size 3 3) (drill 3) (layers *.Cu *.Mask F.SilkS))
+  )
+  (module holemoi:hole (layer F.Cu)
+    (at 621.25 595)
+    (fp_text reference REF** (at 0 0.5) (layer F.SilkS)
+      (effects (font (size 1 1) (thickness 0.15)))
+    )
+    (fp_text value hole (at 0 -0.5) (layer F.Fab)
+      (effects (font (size 1 1) (thickness 0.15)))
+    )
+    (pad 1 thru_hole circle (at 0 0) (size 3 3) (drill 3) (layers *.Cu *.Mask F.SilkS))
+  )
+  (module holemoi:hole (layer F.Cu)
+    (at 853.75 595)
+    (fp_text reference REF** (at 0 0.5) (layer F.SilkS)
+      (effects (font (size 1 1) (thickness 0.15)))
+    )
+    (fp_text value hole (at 0 -0.5) (layer F.Fab)
+      (effects (font (size 1 1) (thickness 0.15)))
+    )
+    (pad 1 thru_hole circle (at 0 0) (size 3 3) (drill 3) (layers *.Cu *.Mask F.SilkS))
+  )
+  (dimension 232.5 (width 0.3) (layer F.Paste)
+    (gr_text "232.500 mm" (at 737.5 541) (layer F.Paste)
+      (effects (font (size 1.5 1.5) (thickness 0.3)))
+    )
+    (feature1 (pts (xy 853.75 541) (xy 853.75 541)))
+    (feature2 (pts (xy 621.25 541) (xy 621.25 541)))
+    (crossbar (pts (xy 621.25 541) (xy 853.75 541)))
+    (arrow1a (pts (xy 853.75 541) (xy 852.623496 541.586421)))
+    (arrow1b (pts (xy 853.75 541) (xy 852.623496 540.413579)))
+    (arrow2a (pts (xy 621.25 541) (xy 622.376504 541.586421)))
+    (arrow2b (pts (xy 621.25 541) (xy 622.376504 540.413579)))
+  )
+  (dimension 116.25 (width 0.3) (layer F.Paste)
+    (gr_text "116.250 mm" (at 98.125 541) (layer F.Paste)
+      (effects (font (size 1.5 1.5) (thickness 0.3)))
+    )
+    (feature1 (pts (xy 156.25 541) (xy 156.25 541)))
+    (feature2 (pts (xy 40 541) (xy 40 541)))
+    (crossbar (pts (xy 40 541) (xy 156.25 541)))
+    (arrow1a (pts (xy 156.25 541) (xy 155.123496 541.586421)))
+    (arrow1b (pts (xy 156.25 541) (xy 155.123496 540.413579)))
+    (arrow2a (pts (xy 40 541) (xy 41.126504 541.586421)))
+    (arrow2b (pts (xy 40 541) (xy 41.126504 540.413579)))
+  )
   (dimension 30 (width 0.3) (layer F.Paste)
     (gr_text "30,000 mm" (at 25.50825 595 270) (layer F.Paste)
@@
   (segment (start 749.527 610) (end 749.527 611.6) (width 0.75) (layer F.Cu) (net 153))
   (segment (start 749.527 608.4) (end 749.527 610) (width 0.75) (layer F.Cu) (net 153))
+  (segment (start 968.8 590) (end 968.8 572.8) (width 1.5) (layer F.Cu) (net 154))
+  (segment (start 273 572) (end 42.7 572) (width 4) (layer F.Cu) (net 154))
+  (segment (start 42.7 572) (end 42.6 572.1) (width 4) (layer F.Cu) (net 154))
+  (segment (start 276.1 618) (end 734.5 618) (width 4) (layer F.Cu) (net 154))
+  (segment (start 734.5 618) (end 736.8 618) (width 4) (layer F.Cu) (net 154))
+  (segment (start 740.1 618) (end 734.5 618) (width 1) (layer F.Cu) (net 154))
+  (segment (start 740.1 618) (end 736.8 618) (width 1) (layer F.Cu) (net 154))
+  (segment (start 740.1 618) (end 737.8 618) (width 1) (layer F.Cu) (net 154))
+  (segment (start 737.8 618) (end 737.7 618.1) (width 1) (layer F.Cu) (net 154))
+  (segment (start 740 618.1) (end 740.1 618) (width 4) (layer F.Cu) (net 154))
+  (segment (start 740.1 618) (end 967.5 618) (width 4) (layer F.Cu) (net 154))
+  (segment (start 967.5 618) (end 967.6 618.1) (width 4) (layer F.Cu) (net 154))
+  (segment (start 737.7 618.1) (end 740 618.1) (width 4) (layer F.Cu) (net 154))
+  (segment (start 730.8 618.1) (end 737.7 618.1) (width 4) (layer F.Cu) (net 154))
+  (segment (start 740 618.1) (end 737.2 618.1) (width 1) (layer F.Cu) (net 154))
+  (segment (start 737.2 618.1) (end 736.9 618.1) (width 1) (layer F.Cu) (net 154))
+  (segment (start 737.7 618.1) (end 737.2 618.1) (width 1) (layer F.Cu) (net 154))
+  (segment (start 736.9 618.1) (end 736.8 618) (width 1) (layer F.Cu) (net 154))
   (segment (start 968.8 618.6) (end 968.1 618.6) (width 1) (layer F.Cu) (net 154))
   (segment (start 968.1 618.6) (end 967.6 618.1) (width 1) (layer F.Cu) (net 154))
@@
   (segment (start 968.8 616) (end 968.8 616.9) (width 1) (layer F.Cu) (net 154))
   (segment (start 968.8 616.9) (end 967.6 618.1) (width 1) (layer F.Cu) (net 154))
-  (segment (start 730.6 617.9) (end 730.8 618.1) (width 4) (layer F.Cu) (net 154))
-  (segment (start 730.8 618.1) (end 967.6 618.1) (width 4) (layer F.Cu) (net 154))
   (segment (start 41.5 595) (end 41.2 595.3) (width 1.5) (layer F.Cu) (net 154))
   (segment (start 41.2 595.3) (end 41.2 617.8) (width 1.5) (layer F.Cu) (net 154))
@@
   (segment (start 42 617.5) (end 42.5 618) (width 0.75) (layer F.Cu) (net 154))
   (segment (start 42.5 618) (end 286 618) (width 4) (layer F.Cu) (net 154))
-  (segment (start 276.1 618) (end 736.8 618) (width 4) (layer F.Cu) (net 154))
   (segment (start 967.8 572) (end 737.3 572) (width 4) (layer F.Cu) (net 154))
   (segment (start 737.55 583.85) (end 737.55 572.25) (width 0.75) (layer F.Cu) (net 154))
@@
   (segment (start 272.5 573.1) (end 272.4 573) (width 0.75) (layer F.Cu) (net 154))
   (segment (start 275 583.8) (end 272.5 583.8) (width 0.75) (layer F.Cu) (net 154))
-  (segment (start 270 573) (end 42.5 573) (width 4) (layer F.Cu) (net 154))
   (segment (start 270 576.15) (end 270 573) (width 0.75) (layer F.Cu) (net 154))
-  (segment (start 42.5 573) (end 42.4 573.1) (width 4) (layer F.Cu) (net 154))
-  (segment (start 968.8 590) (end 969 589.8) (width 1.5) (layer F.Cu) (net 154))
-  (segment (start 969 589.8) (end 969 573) (width 1.5) (layer F.Cu) (net 154))
-  (segment (start 969 573) (end 968.8 572.8) (width 1.5) (layer F.Cu) (net 154))
   (segment (start 968.8 572.8) (end 967.299998 572.8) (width 0.75) (layer F.Cu) (net 154))
   (segment (start 967.299998 572.8) (end 967.149999 572.949999) (width 0.75) (layer F.Cu) (net 154))
@@
   (segment (start 463.907 580) (end 487.969 580) (width 0.75) (layer F.Cu) (net 194))
   (segment (start 463.907 578.4) (end 487.969 578.4) (width 0.75) (layer F.Cu) (net 195))
+  (zone (net 0) (net_name "") (layer F.Mask) (hatch edge 0.508)
+    (connect_pads (clearance 0.508))
+    (min_thickness 0.254)
+    (fill yes (arc_segments 16) (thermal_gap 0.508) (thermal_bridge_width 0.508))
+    (polygon
+      (pts
+        (xy 962.3 576.2) (xy 967.1 576.2) (xy 967 583.8) (xy 962.3 583.8)
+      )
+    )
+  )
+  (zone (net 0) (net_name "") (layer F.Mask) (hatch edge 0.508)
+    (connect_pads (clearance 0.508))
+    (min_thickness 0.254)
+    (fill yes (arc_segments 16) (thermal_gap 0.508) (thermal_bridge_width 0.508))
+    (polygon
+      (pts
+        (xy 962.3 591.2) (xy 967.1 591.2) (xy 967.1 598.8) (xy 962.3 598.8)
+      )
+    )
+  )
+  (zone (net 0) (net_name "") (layer F.Mask) (hatch edge 0.508)
+    (connect_pads (clearance 0.508))
+    (min_thickness 0.254)
+    (fill yes (arc_segments 16) (thermal_gap 0.508) (thermal_bridge_width 0.508))
+    (polygon
+      (pts
+        (xy 962.4 606.2) (xy 967.2 606.2) (xy 967.2 613.8) (xy 962.4 613.8)
+      )
+    )
+  )
+  (zone (net 0) (net_name "") (layer F.Mask) (hatch edge 0.508)
+    (connect_pads (clearance 0.508))
+    (min_thickness 0.254)
+    (fill yes (arc_segments 16) (thermal_gap 0.508) (thermal_bridge_width 0.508))
+    (polygon
+      (pts
+        (xy 47.8 576.2) (xy 43 576.2) (xy 43 583.7) (xy 47.7 583.8)
+      )
+    )
+  )
+  (zone (net 0) (net_name "") (layer F.Mask) (hatch edge 0.508)
+    (connect_pads (clearance 0.508))
+    (min_thickness 0.254)
+    (fill yes (arc_segments 16) (thermal_gap 0.508) (thermal_bridge_width 0.508))
+    (polygon
+      (pts
+        (xy 43 591.2) (xy 47.8 591.2) (xy 47.7 598.8) (xy 43 598.9)
+      )
+    )
+  )
+  (zone (net 0) (net_name "") (layer F.Mask) (hatch edge 0.508)
+    (connect_pads (clearance 0.508))
+    (min_thickness 0.254)
+    (fill yes (arc_segments 16) (thermal_gap 0.508) (thermal_bridge_width 0.508))
+    (polygon
+      (pts
+        (xy 43 606.26) (xy 47.79 606.24) (xy 47.9 613.74) (xy 43 613.72)
+      )
+    )
+  )
+  (zone (net 154) (net_name GND) (layer F.Cu) (hatch edge 0.508)
+    (connect_pads (clearance 1.2))
+    (min_thickness 0.254)
+    (fill yes (arc_segments 16) (thermal_gap 0.508) (thermal_bridge_width 0.508))
+    (polygon
+      (pts
+        (xy 40 570) (xy 969.9 570) (xy 970 620) (xy 40 620)
+      )
+    )
+  )
 )
